File: box0-interface.sch (KiCad schematic (older format))
At the start: 2 parts, among them P2 BASE_BOARD_ANALOG, P3 BASE_BOARD_DIGITAL

Commit message: fixed the wrongly connected VREF
Connections:
- net GND: now also P2.7 (P7); no longer P2.8 (P8)
- net VREF_EXT: now also P2.8 (P8); no longer P2.7 (P7)
Changed lines of the file:
@@
 Text GLabel 3550 2650 0    60   Output ~ 0
 ANALOG_NEG
-Text GLabel 4050 2850 2    60   Output ~ 0
+Text GLabel 3500 2850 0    60   Output ~ 0
 VREF_EXT
 Wire Wire Line
@@
 	3550 3350 2950 3350
 Connection ~ 2950 3350
-Wire Wire Line
-	3550 2850 2950 2850
 Connection ~ 2950 2850
 Wire Wire Line
 	4050 3750 4800 3750
 Connection ~ 4800 3750
+Wire Wire Line
+	3550 2850 3500 2850
+Wire Wire Line
+	4050 2850 4800 2850
 $EndSCHEMATC
