File: breakout.kicad_pcb (KiCad board)
At the start: 2 copper layers, 70 x 50 mm, 5 parts, among them P2 BASE_BOARD_ANALOG, P3 BASE_BOARD_DIGITAL

Commit message: Schematic nearly done
Parts:
- added P1: USB_OTG, Connect:USB_Micro-B, F.Cu at (108.2, 54.2)
Changed lines of the file:
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@@
 (kicad_pcb (version 4) (host pcbnew 4.0.2+dfsg1-stable)
   (general
-    (links 26)
+    (links 31)
     (no_connects 0)
-    (area 57.979681 27.19852 203.228501 150.760441)
+    (area 90.831499 50.348519 160.931501 100.448521)
     (thickness 1.6)
     (drawings 28)
     (tracks 6)
     (zones 0)
-    (modules 5)
+    (modules 6)
     (nets 5)
   )
@@
   )
   (setup
-    (last_trace_width 0.25)
+    (last_trace_width 0.2)
     (user_trace_width 0.2)
     (user_trace_width 0.25)
@@
     )
   )
+  (module Connect:USB_Micro-B (layer F.Cu)
+    (at 108.1535 54.20852 180)
+    (descr "Micro USB Type B Receptacle")
+    (tags "USB USB_B USB_micro USB_OTG")
+    (attr smd)
+    (fp_text reference P1 (at 0 -3.45 180) (layer F.SilkS)
+      (effects (font (size 1 1) (thickness 0.15)))
+    )
+    (fp_text value USB_OTG (at 0 4.8 180) (layer F.Fab)
+      (effects (font (size 1 1) (thickness 0.15)))
+    )
+    (fp_line (start -4.6 -2.8) (end 4.6 -2.8) (layer F.CrtYd) (width 0.05))
+    (fp_line (start 4.6 -2.8) (end 4.6 4.05) (layer F.CrtYd) (width 0.05))
+    (fp_line (start 4.6 4.05) (end -4.6 4.05) (layer F.CrtYd) (width 0.05))
+    (fp_line (start -4.6 4.05) (end -4.6 -2.8) (layer F.CrtYd) (width 0.05))
+    (fp_line (start -4.3509 3.81746) (end 4.3491 3.81746) (layer F.SilkS) (width 0.15))
+    (fp_line (start -4.3509 -2.58754) (end 4.3491 -2.58754) (layer F.SilkS) (width 0.15))
+    (fp_line (start 4.3491 -2.58754) (end 4.3491 3.81746) (layer F.SilkS) (width 0.15))
+    (fp_line (start 4.3491 2.58746) (end -4.3509 2.58746) (layer F.SilkS) (width 0.15))
+    (fp_line (start -4.3509 3.81746) (end -4.3509 -2.58754) (layer F.SilkS) (width 0.15))
+    (pad 1 smd rect (at -1.3009 -1.56254 270) (size 1.35 0.4) (layers F.Cu F.Paste F.Mask))
+    (pad 2 smd rect (at -0.6509 -1.56254 270) (size 1.35 0.4) (layers F.Cu F.Paste F.Mask))
+    (pad 3 smd rect (at -0.0009 -1.56254 270) (size 1.35 0.4) (layers F.Cu F.Paste F.Mask))
+    (pad 4 smd rect (at 0.6491 -1.56254 270) (size 1.35 0.4) (layers F.Cu F.Paste F.Mask))
+    (pad 5 smd rect (at 1.2991 -1.56254 270) (size 1.35 0.4) (layers F.Cu F.Paste F.Mask)
+      (net 3 GND))
+    (pad 6 thru_hole oval (at -2.5009 -1.56254 270) (size 0.95 1.25) (drill oval 0.55 0.85) (layers *.Cu *.Mask F.SilkS)
+      (net 3 GND))
+    (pad 6 thru_hole oval (at 2.4991 -1.56254 270) (size 0.95 1.25) (drill oval 0.55 0.85) (layers *.Cu *.Mask F.SilkS)
+      (net 3 GND))
+    (pad 6 thru_hole oval (at -3.5009 1.13746 270) (size 1.55 1) (drill oval 1.15 0.5) (layers *.Cu *.Mask F.SilkS)
+      (net 3 GND))
+    (pad 6 thru_hole oval (at 3.4991 1.13746 270) (size 1.55 1) (drill oval 1.15 0.5) (layers *.Cu *.Mask F.SilkS)
+      (net 3 GND))
+  )
   (gr_line (start 141.872 62.28318) (end 141.872 57.18794) (angle 90) (layer Cmts.User) (width 0.001))

Commit message: Started on PCB
Parts:
- added C10: 100n, rik_footprints:0603, F.Cu at (245.9, 96.6)
- added C11: 100n, rik_footprints:0603, F.Cu at (246.6, 79.6)
- added C12: 100n, rik_footprints:0603, F.Cu at (256.5, 94.1)
- added C13: 100n, rik_footprints:0603, F.Cu at (257.0, 77.1)
- added C14: 100n, rik_footprints:0603, F.Cu at (191.5, 113.1)
- added C4: 4.7u, rik_footprints:0805, F.Cu at (191.8, 95.5)
- added C5: 4.7u, rik_footprints:0805, F.Cu at (192.0, 83.4)
- added C6: 82p, rik_footprints:0603, F.Cu at (202.0, 92.9)
- added C7: 82p, rik_footprints:0603, F.Cu at (202.1, 80.4)
- added C8: 10u, rik_footprints:0805, F.Cu at (203.3, 96.1)
- added C9: 10u, rik_footprints:0805, F.Cu at (203.4, 84.2)
- added D1: MBR0540, Diodes_SMD:SOD-123, F.Cu at (199.5, 95.5)
- added D2: MBR0540, Diodes_SMD:SOD-123, F.Cu at (199.6, 83.5)
- added IC1: LM2733, TO_SOT_Packages_SMD:SOT-23-5, F.Cu at (195.0, 92.3)
- added IC2: LM2733, TO_SOT_Packages_SMD:SOT-23-5, F.Cu at (195.1, 80.1)
- added IC3: OPA454, rik_footprints:SOIC-8-3.9*4.9mm_HP_to_P4, F.Cu at (251.0, 94.8)
- added IC4: OPA454, rik_footprints:SOIC-8-3.9*4.9mm_HP_to_P4, F.Cu at (251.7, 77.8)
- added JP1: Jumper_NO_Small, Capacitors_SMD:C_0201, F.Cu at (185.1, 119.0)
- added L1: 10u, rik_footprints:0805, F.Cu at (195.0, 95.5)
- added L2: 10u, rik_footprints:0805, F.Cu at (195.1, 83.5)
- added P4: CONN_02X04, Pin_Headers:Pin_Header_Straight_2x04, F.Cu at (270.0, 90.8)
- added P5: CONN_01X04, Pin_Headers:Pin_Header_Straight_1x04, F.Cu at (186.1, 134.7)
- added P6: CONN_01X04, Pin_Headers:Pin_Header_Straight_1x04, F.Cu at (186.1, 132.2)
- added P7: CONN_01X04, Pin_Headers:Pin_Header_Straight_1x04, F.Cu at (186.1, 129.6)
- added P8: CONN_01X04, Pin_Headers:Pin_Header_Straight_1x04, F.Cu at (186.1, 127.1)
- added R1: 47K, rik_footprints:0603, F.Cu at (192.5, 92.3)
- added R10: 91K, rik_footprints:0603, F.Cu at (250.9, 98.4)
- added R11: 1M, rik_footprints:0603, F.Cu at (257.0, 75.5)
- added R12: 91K, rik_footprints:0603, F.Cu at (251.7, 81.4)
- added R13: 10R, rik_footprints:0603, F.Cu at (256.5, 95.6)
- added R14: 10R, rik_footprints:0603, F.Cu at (257.0, 78.6)
- added R15: 91K, rik_footprints:0603, F.Cu at (187.1, 123.8)
- added R16: 10K, rik_footprints:0603, F.Cu at (185.6, 123.8)
- added R17: 91K, rik_footprints:0603, F.Cu at (181.1, 123.8)
- added R18: 10K, rik_footprints:0603, F.Cu at (179.5, 123.8)
- added R19: 4.7K, rik_footprints:0603, F.Cu at (180.0, 113.9)
- added R2: 47K, rik_footprints:0603, F.Cu at (192.6, 80.1)
- added R20: 91K, rik_footprints:0603, F.Cu at (184.1, 123.8)
- added R21: 10K, rik_footprints:0603, F.Cu at (182.6, 123.8)
- added R22: 91K, rik_footprints:0603, F.Cu at (178.0, 123.8)
- added R23: 10K, rik_footprints:0603, F.Cu at (176.5, 123.8)
- added R24: 4.7K, rik_footprints:0603, F.Cu at (181.8, 114.7)
- added R3: 12K, rik_footprints:0603, F.Cu at (198.2, 91.7)
- added R4: 12K, rik_footprints:0603, F.Cu at (198.3, 79.1)
- added R5: 309K, rik_footprints:0603, F.Cu at (200.1, 92.9)
- added R6: 309K, rik_footprints:0603, F.Cu at (200.2, 80.4)
- added R7: 10K, rik_footprints:0603, F.Cu at (245.8, 94.3)
- added R8: 10K, rik_footprints:0603, F.Cu at (246.6, 77.3)
- added R9: 1M, rik_footprints:0603, F.Cu at (256.5, 92.6)
- added U1: 24C16, Housings_SOIC:SOIC-8_3.9x4.9mm_Pitch1.27mm, F.Cu at (186.6, 114.4)
- C1, C2, C3: footprint Capacitors_SMD:C_0603_HandSoldering -> rik_footprints:0603
Connections:
- P1 pad 1: (no net) -> 5V
- P2 pad 12: (no net) -> /Box0 Interface/AOUT0.0
- P2 pad 14: (no net) -> /Box0 Interface/AOUT0.1
- P2 pad 20: (no net) -> /Box0 Interface/AIN0.0
- P2 pad 22: (no net) -> /Box0 Interface/AIN0.1
- P2 pad 24: (no net) -> /Box0 Interface/AIN0.2
- P2 pad 26: (no net) -> /Box0 Interface/AIN0.3
- P3 pad 24: (no net) -> /Box0 Interface/I2C0.SCL
- P3 pad 25: (no net) -> DIGITAL_EXT
- P3 pad 26: (no net) -> /Box0 Interface/I2C0.SDA

Commit message: PCB almost done
Parts:
- moved P4 126.8 mm to (145.2, 67.7)
- moved C12 118.8 mm to (140.2, 70.0)
- moved R10 118.8 mm to (134.6, 74.3)
- moved R13 118.8 mm to (140.2, 71.5)
- moved R9 118.8 mm to (140.1, 68.4)
- moved C10 118.8 mm to (129.5, 72.5)
- moved IC3 118.8 mm to (134.6, 70.6)
- moved R7 118.8 mm to (129.5, 70.2)
- moved C13 118.1 mm to (140.2, 59.8)
- moved IC4 118.1 mm to (134.8, 60.6)
- moved R11 118.1 mm to (140.1, 58.3)
- moved R12 118.1 mm to (134.8, 64.1)
- moved R14 118.1 mm to (140.2, 61.3)
- moved C11 118.1 mm to (129.7, 62.3)
- moved R8 118.1 mm to (129.7, 60.1)
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Routing:
- net /Box0 Interface/AOUT0.0: track 0.00 -> 43.5 mm, vias 0 -> 2
- net /Box0 Interface/AOUT0.1: track 0.00 -> 34.3 mm, vias 0 -> 2
- net 5V: track 0.00 -> 32.5 mm
- net /Box0 Interface/AIN0.0: track 0.00 -> 21.1 mm
- net /Box0 Interface/AIN0.1: track 0.00 -> 18.8 mm
- net -33V: track 0.00 -> 18.2 mm
- net /Box0 Interface/AIN0.2: track 0.00 -> 16.7 mm
- net +33V: track 0.00 -> 14.3 mm
- net /Box0 Interface/AIN0.3: track 0.00 -> 14.2 mm
- net Net-(IC3-Pad2): track 0.00 -> 10.2 mm
- net Net-(IC4-Pad2): track 0.00 -> 10.0 mm
- net Net-(P4-Pad1): track 0.00 -> 9.59 mm
- net Net-(P4-Pad2): track 0.00 -> 9.14 mm
- net Net-(C7-Pad1): track 0.00 -> 8.86 mm
- net Net-(IC3-Pad6): track 0.00 -> 8.41 mm
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
Commit message: Finished PCB
Parts:
- added F1: F_Small, SMD_Packages:SMD-1210_Pol, F.Cu at (106.4, 61.8)
- moved C1 7.03 mm to (159.7, 66.6)
Connections:
- P1 pad 1: 5V -> Net-(F1-Pad2)
Routing:
- net +33V: track 14.3 -> 92.0 mm, vias 0 -> 4
- net -33V: track 18.2 -> 72.2 mm, vias 0 -> 2
- net DIGITAL_EXT: track 0.00 -> 34.4 mm, vias 0 -> 1
- net /Box0 Interface/I2C0.SCL: track 2.16 -> 23.5 mm
- net /Box0 Interface/I2C0.SDA: track 4.15 -> 15.1 mm
- net Net-(F1-Pad2): track 0.00 -> 7.78 mm
- net Net-(JP1-Pad2): track 0.00 -> 5.14 mm
- net VREF_EXT: track 5.35 -> 2.21 mm
- net 5V: track 32.5 -> 30.0 mm
- added copper zone on F.Cu, net -33V
Other:
- board text added: "AIN !HV!"
- board text added: "AOUT !HV!"
- board text added: "CH0"
- board text added: "CH1"
- board text added: "CHx -33V +33V GND"
- board text added: "CHx GND GND GND"

Commit message: fixed the wrongly connected VREF
Parts:
- moved C1 6.94 mm to (152.9, 67.7)
Connections:
- P2 pad 7: VREF_EXT -> GND
- P2 pad 8: GND -> VREF_EXT
Routing:
- net GND: track 0.00 -> 0.51 mm
Changed lines of the file:
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@@
   (general
     (links 155)
-    (no_connects 25)
+    (no_connects 0)
     (area 90.831499 50.348519 160.931501 100.448521)
     (thickness 1.6)
     (drawings 34)
-    (tracks 276)
+    (tracks 278)
     (zones 0)
     (modules 57)
@@
   )
   (setup
-    (last_trace_width 0.8)
+    (last_trace_width 0.4)
     (user_trace_width 0.2)
     (user_trace_width 0.25)
@@
   )
   (module rik_footprints:0603 (layer F.Cu)
-    (at 159.7155 66.61652 90)
+    (at 152.8575 67.67052 90)
     (descr "Resistor SMD 0603, reflow soldering, Vishay (see dcrcw.pdf)")
     (tags "resistor 0603")
@@
       (net 3 GND))
     (pad 7 thru_hole oval (at 0 -7.62 180) (size 1.7272 1.7272) (drill 1.016) (layers *.Cu *.Mask B.SilkS)
+      (net 3 GND))
+    (pad 8 thru_hole oval (at 2.54 -7.62 180) (size 1.7272 1.7272) (drill 1.016) (layers *.Cu *.Mask B.SilkS)
       (net 4 VREF_EXT))
-    (pad 8 thru_hole oval (at 2.54 -7.62 180) (size 1.7272 1.7272) (drill 1.016) (layers *.Cu *.Mask B.SilkS)
-      (net 3 GND))
     (pad 9 thru_hole oval (at 0 -10.16 180) (size 1.7272 1.7272) (drill 1.016) (layers *.Cu *.Mask B.SilkS)
       (net 3 GND))
@@
   (segment (start 152.8575 63.67252) (end 154.14024 63.67252) (width 0.25) (layer F.Cu) (net 2))
   (segment (start 154.14024 63.67252) (end 155.11302 62.69974) (width 0.25) (layer F.Cu) (net 2))
-  (segment (start 159.7155 67.41652) (end 158.01624 67.41652) (width 0.4) (layer F.Cu) (net 4))
-  (segment (start 158.01624 67.41652) (end 157.65302 67.77974) (width 0.4) (layer F.Cu) (net 4))
+  (segment (start 158.01624 67.41652) (end 157.65302 67.77974) (width 0.4) (layer F.Cu) (net 3))
+  (segment (start 155.03428 67.77974) (end 154.3435 68.47052) (width 0.4) (layer F.Cu) (net 4))
+  (segment (start 154.3435 68.47052) (end 152.8575 68.47052) (width 0.4) (layer F.Cu) (net 4))
+  (segment (start 155.11302 67.77974) (end 155.03428 67.77974) (width 0.4) (layer F.Cu) (net 4))
   (segment (start 109.4544 61.32052) (end 109.4544 63.60652) (width 0.8) (layer F.Cu) (net 5))
   (segment (start 109.4544 63.60652) (end 109.4544 68.97142) (width 0.8) (layer F.Cu) (net 5))
